Commit message: update robot_controller

File: robot_description/urdf/bot.xacro (robot description, xacro)
@@ -65,8 +65,8 @@
     <origin xyz="${body_length/2 - 0.025} 0 0.1" rpy="0 ${0 * pi/180.0} 0"/>
     <parent link="base_link"/>
-    <child link="camera_link"/>
+    <child link="bot_camera_link"/>
   </joint>
   <!-- Camera -->
-  <link name="camera_link">
+  <link name="bot_camera_link">
     <collision>
       <origin xyz="0 0 0" rpy="0 0 0"/>

File: robot_description/urdf/gazebo.xacro (robot description, xacro)
@@ -61,3 +61,42 @@
     </sensor>
   </gazebo>
+  <gazebo reference="bot_camera_link">
+    <sensor type="camera" name="camera1">
+      <update_rate>5.0</update_rate>
+      <camera name="head">
+        <horizontal_fov>1.3962634</horizontal_fov>
+        <image>
+          <width>800</width>
+          <height>800</height>
+          <format>R8G8B8</format>
+        </image>
+        <clip>
+          <near>0.02</near>
+          <far>3</far>
+        </clip>
+        <noise>
+          <type>gaussian</type>
+          <!-- Noise is sampled independently per pixel on each frame.
+               That pixel's noise value is added to each of its color
+               channels, which at that point lie in the range [0,1]. -->
+          <mean>0.0</mean>
+          <stddev>0.007</stddev>
+        </noise>
+      </camera>
+      <plugin name="camera_controller" filename="libgazebo_ros_camera.so">
+        <alwaysOn>true</alwaysOn>
+        <updateRate>0.0</updateRate>
+        <cameraName>camera</cameraName>
+        <imageTopicName>image_raw</imageTopicName>
+        <cameraInfoTopicName>camera_info</cameraInfoTopicName>
+        <frameName>camera_link</frameName>
+        <hackBaseline>0.07</hackBaseline>
+        <distortionK1>0.0</distortionK1>
+        <distortionK2>0.0</distortionK2>
+        <distortionK3>0.0</distortionK3>
+        <distortionT1>0.0</distortionT1>
+        <distortionT2>0.0</distortionT2>
+      </plugin>
+    </sensor>
+  </gazebo>
 </robot>
